File: PCBs Taller KiCad/FuenteAlimentacionDual/FuenteAlimentacionDual.kicad_pcb (KiCad board)
At the start: 2 copper layers, 130.5 x 80 mm, 28 parts, among them J1 Conn_01x03, J2 Conn_01x03, U1 LM317_TO-220, U2 LM337_TO220

Commit message: modification
Connections:
- D5 pad 1: VOUT+ -> VIN+
- D5 pad 2: VIN+ -> VOUT+
- D6 pad 1: VIN- -> VOUT-
- D6 pad 2: VOUT- -> VIN-
Changed lines of the file:
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@@
 		(property ki_fp_filters "TO?220*")
 		(sheetname "/")
-		(sheetfile "Fuente de alimentación dual ajustable ±1.25V a ±12V.kicad_sch")
+		(sheetfile "FuenteAlimentacionDual.kicad_sch")
 		(units
 			(unit
@@
 		(property ki_fp_filters "LED* LED_SMD:* LED_THT:*")
 		(sheetname "/")
-		(sheetfile "Fuente de alimentación dual ajustable ±1.25V a ±12V.kicad_sch")
+		(sheetfile "FuenteAlimentacionDual.kicad_sch")
 		(units
 			(unit
@@
 		(property ki_fp_filters "CP_*")
 		(sheetname "/")
-		(sheetfile "Fuente de alimentación dual ajustable ±1.25V a ±12V.kicad_sch")
+		(sheetfile "FuenteAlimentacionDual.kicad_sch")
 		(units
 			(unit
@@
 		(property ki_fp_filters "D*DO?41*")
 		(sheetname "/")
-		(sheetfile "Fuente de alimentación dual ajustable ±1.25V a ±12V.kicad_sch")
+		(sheetfile "FuenteAlimentacionDual.kicad_sch")
 		(units
 			(unit
@@
 			(remove_unused_layers no)
 			(roundrect_rratio 0.113636)
-			(net "VOUT+")
+			(net "VIN+")
 			(pinfunction "K_1")
 			(pintype "passive")
@@
 			(layers "*.Cu" "*.Mask")
 			(remove_unused_layers no)
-			(net "VIN+")
+			(net "VOUT+")
 			(pinfunction "A_2")
 			(pintype "passive")
@@
 		(property ki_fp_filters "D*DO?41*")
 		(sheetname "/")
-		(sheetfile "Fuente de alimentación dual ajustable ±1.25V a ±12V.kicad_sch")
+		(sheetfile "FuenteAlimentacionDual.kicad_sch")
 		(units
 			(unit
@@
 		(property ki_fp_filters "R_*")
 		(sheetname "/")
-		(sheetfile "Fuente de alimentación dual ajustable ±1.25V a ±12V.kicad_sch")
+		(sheetfile "FuenteAlimentacionDual.kicad_sch")
 		(units
 			(unit
@@
 		(property ki_fp_filters "CP_*")
 		(sheetname "/")
-		(sheetfile "Fuente de alimentación dual ajustable ±1.25V a ±12V.kicad_sch")
+		(sheetfile "FuenteAlimentacionDual.kicad_sch")
 		(units
 			(unit
@@
 		(property ki_fp_filters "R_*")
 		(sheetname "/")
-		(sheetfile "Fuente de alimentación dual ajustable ±1.25V a ±12V.kicad_sch")
+		(sheetfile "FuenteAlimentacionDual.kicad_sch")
 		(units
 			(unit
@@
 		(property ki_fp_filters "C_*")
 		(sheetname "/")
-		(sheetfile "Fuente de alimentación dual ajustable ±1.25V a ±12V.kicad_sch")
+		(sheetfile "FuenteAlimentacionDual.kicad_sch")
 		(units
 			(unit
@@
 		(property ki_fp_filters "D*DO?41*")
 		(sheetname "/")
-		(sheetfile "Fuente de alimentación dual ajustable ±1.25V a ±12V.kicad_sch")
+		(sheetfile "FuenteAlimentacionDual.kicad_sch")
 		(units
 			(unit
@@
 			(remove_unused_layers no)
 			(roundrect_rratio 0.113636)
-			(net "VIN-")
+			(net "VOUT-")
 			(pinfunction "K_1")
 			(pintype "passive")
@@
 			(layers "*.Cu" "*.Mask")
 			(remove_unused_layers no)
-			(net "VOUT-")
+			(net "VIN-")
 			(pinfunction "A_2")
 			(pintype "passive")
@@
 		(property ki_fp_filters "CP_*")
 		(sheetname "/")
-		(sheetfile "Fuente de alimentación dual ajustable ±1.25V a ±12V.kicad_sch")
+		(sheetfile "FuenteAlimentacionDual.kicad_sch")
 		(units
 			(unit
@@
 		(property ki_fp_filters "TO?220*")
 		(sheetname "/")
-		(sheetfile "Fuente de alimentación dual ajustable ±1.25V a ±12V.kicad_sch")
+		(sheetfile "FuenteAlimentacionDual.kicad_sch")
 		(units
 			(unit
@@
 		(property ki_fp_filters "C_*")
 		(sheetname "/")
-		(sheetfile "Fuente de alimentación dual ajustable ±1.25V a ±12V.kicad_sch")
+		(sheetfile "FuenteAlimentacionDual.kicad_sch")
 		(units
 			(unit
@@
 		(property ki_fp_filters "CP_*")
 		(sheetname "/")
-		(sheetfile "Fuente de alimentación dual ajustable ±1.25V a ±12V.kicad_sch")
+		(sheetfile "FuenteAlimentacionDual.kicad_sch")
 		(units
 			(unit
@@
 		(property ki_fp_filters "R_*")
 		(sheetname "/")
-		(sheetfile "Fuente de alimentación dual ajustable ±1.25V a ±12V.kicad_sch")
+		(sheetfile "FuenteAlimentacionDual.kicad_sch")
 		(units
 			(unit
@@
 		(property ki_fp_filters "D*DO?41*")
 		(sheetname "/")
-		(sheetfile "Fuente de alimentación dual ajustable ±1.25V a ±12V.kicad_sch")
+		(sheetfile "FuenteAlimentacionDual.kicad_sch")
 		(units
 			(unit
@@
 		(property ki_fp_filters "Connector*:*_1x??_*")
 		(sheetname "/")
-		(sheetfile "Fuente de alimentación dual ajustable ±1.25V a ±12V.kicad_sch")
+		(sheetfile "FuenteAlimentacionDual.kicad_sch")
 		(units
 			(unit
@@
 		(property ki_fp_filters "Connector*:*_1x??_*")
 		(sheetname "/")
-		(sheetfile "Fuente de alimentación dual ajustable ±1.25V a ±12V.kicad_sch")
+		(sheetfile "FuenteAlimentacionDual.kicad_sch")
 		(units
 			(unit
@@
 		(property ki_fp_filters "R_*")
 		(sheetname "/")
-		(sheetfile "Fuente de alimentación dual ajustable ±1.25V a ±12V.kicad_sch")
+		(sheetfile "FuenteAlimentacionDual.kicad_sch")
 		(units
 			(unit
@@
 		(property ki_fp_filters "D*DO?41*")
 		(sheetname "/")
-		(sheetfile "Fuente de alimentación dual ajustable ±1.25V a ±12V.kicad_sch")
+		(sheetfile "FuenteAlimentacionDual.kicad_sch")
 		(units
 			(unit
@@
 		(property ki_fp_filters "Potentiometer*")
 		(sheetname "/")
-		(sheetfile "Fuente de alimentación dual ajustable ±1.25V a ±12V.kicad_sch")
+		(sheetfile "FuenteAlimentacionDual.kicad_sch")
 		(units
 			(unit
@@
 		(property ki_fp_filters "Potentiometer*")
 		(sheetname "/")
-		(sheetfile "Fuente de alimentación dual ajustable ±1.25V a ±12V.kicad_sch")
+		(sheetfile "FuenteAlimentacionDual.kicad_sch")
 		(units
 			(unit
@@
 		(property ki_fp_filters "D*DO?41*")
 		(sheetname "/")
-		(sheetfile "Fuente de alimentación dual ajustable ±1.25V a ±12V.kicad_sch")
+		(sheetfile "FuenteAlimentacionDual.kicad_sch")
 		(units
 			(unit
@@
 		(property ki_fp_filters "LED* LED_SMD:* LED_THT:*")
 		(sheetname "/")
-		(sheetfile "Fuente de alimentación dual ajustable ±1.25V a ±12V.kicad_sch")
+		(sheetfile "FuenteAlimentacionDual.kicad_sch")
 		(units
 			(unit
