File: PCBs Taller KiCad/LM317_Regulator/LM317_Regulator.kicad_pcb (KiCad board)
At the start: 2 copper layers, 50 x 30 mm, 4 parts

Commit message: Actualización
Parts:
- added C1: C, Capacitor_THT:C_Disc_D5.0mm_W2.5mm_P5.00mm, F.Cu at (68.5, 21.0)
- added C2: C_Polarized, Capacitor_THT:CP_Radial_D5.0mm_P2.50mm, F.Cu at (81.2, 7.00)
- added C3: C_Polarized, Capacitor_THT:CP_Radial_D5.0mm_P2.50mm, F.Cu at (80.8, 16.6)
- added D1: D, Diode_THT:D_DO-41_SOD81_P10.16mm_Horizontal, F.Cu at (71.3, 3.20)
- added D2: D, Diode_THT:D_DO-41_SOD81_P10.16mm_Horizontal, F.Cu at (58.1, 2.54)
- added D3: D, Diode_THT:D_DO-41_SOD81_P10.16mm_Horizontal, F.Cu at (75.1, 17.3)
- added J1: Screw_Terminal_01x02, TerminalBlock_Phoenix:TerminalBlock_Phoenix_MKDS-1,5-2-5.08_1x02_P5.08mm_Horizontal, F.Cu at (57.0, 8.00)
- added J2: Screw_Terminal_01x02, TerminalBlock_Phoenix:TerminalBlock_Phoenix_MKDS-1,5-2-5.08_1x02_P5.08mm_Horizontal, F.Cu at (92.8, 13.5)
- added R1: R_US, Resistor_THT:R_Axial_DIN0207_L6.3mm_D2.5mm_P10.16mm_Horizontal, F.Cu at (71.4, -1.60)
- added RV1: R_Potentiometer_Trim_US, Potentiometer_THT:Potentiometer_Bourns_3296W_Vertical, F.Cu at (86.0, -0.10)
- added U1: LM317_TO-252, Package_TO_SOT_SMD:TO-252-2, F.Cu at (69.8, 10.6)

Commit message: Modificación
Parts:
- removed C1: C, Capacitor_THT:C_Disc_D5.0mm_W2.5mm_P5.00mm
- removed C2, C3: C_Polarized, Capacitor_THT:CP_Radial_D5.0mm_P2.50mm
- removed D1, D2, D3: D, Diode_THT:D_DO-41_SOD81_P10.16mm_Horizontal
- removed J1, J2: Screw_Terminal_01x02, TerminalBlock_Phoenix:TerminalBlock_Phoenix_MKDS-1,5-2-5.08_1x02_P5.08mm_Horizontal
- removed R1: R_US, Resistor_THT:R_Axial_DIN0207_L6.3mm_D2.5mm_P10.16mm_Horizontal
- removed RV1: R_Potentiometer_Trim_US, Potentiometer_THT:Potentiometer_Bourns_3296W_Vertical
- removed U1: LM317_TO-252, Package_TO_SOT_SMD:TO-252-2

Commit message: modification
Parts:
- added C1: C, Capacitor_THT:C_Disc_D5.0mm_W2.5mm_P5.00mm, F.Cu at (68.5, 21.0)
- added C2: C_Polarized, Capacitor_THT:CP_Radial_D5.0mm_P2.50mm, F.Cu at (81.2, 7.00)
- added C3: C_Polarized, Capacitor_THT:CP_Radial_D5.0mm_P2.50mm, F.Cu at (80.8, 16.6)
- added D1: D, Diode_THT:D_DO-41_SOD81_P10.16mm_Horizontal, F.Cu at (71.3, 3.20)
- added D2: D, Diode_THT:D_DO-41_SOD81_P10.16mm_Horizontal, F.Cu at (58.1, 2.54)
- added D3: D, Diode_THT:D_DO-41_SOD81_P10.16mm_Horizontal, F.Cu at (75.1, 17.3)
- added J1: Screw_Terminal_01x02, TerminalBlock_Phoenix:TerminalBlock_Phoenix_MKDS-1,5-2-5.08_1x02_P5.08mm_Horizontal, F.Cu at (57.0, 8.00)
- added J2: Screw_Terminal_01x02, TerminalBlock_Phoenix:TerminalBlock_Phoenix_MKDS-1,5-2-5.08_1x02_P5.08mm_Horizontal, F.Cu at (92.8, 13.5)
- added R1: R_US, Resistor_THT:R_Axial_DIN0207_L6.3mm_D2.5mm_P10.16mm_Horizontal, F.Cu at (71.4, -1.60)
- added RV1: R_Potentiometer_Trim_US, Potentiometer_THT:Potentiometer_Bourns_3296W_Vertical, F.Cu at (86.0, -0.10)
- added U1: LM317_TO-252, Package_TO_SOT_SMD:TO-252-2, F.Cu at (69.8, 10.6)
Routing:
- added copper zone on F.Cu, net GND
